Commit message: feat(twin): 실제 CAD 메시 통합 + 드라이브 축·URDF 영점 확정
Unity Voron24Twin 씬을 실제 CAD 비주얼 메시로 구동하고, 노즐 기준
영점과 조인트 드라이브 축을 확정한 뒤 URDF 파라미터를 동기화한다.

- 씬: fixed_parts/gantry_frame/Y_beam/X_Carriage OBJ 로 mock 박스 대체,
  노즐 월드 (0.1264,0.1433,-0.0869) 를 영점으로 확정
- ArticulationBody 드라이브 축 수정 (메시 재배향 없이 앵커만):
  joint_x(toolhead)→좌우(빔 따라), joint_y(x_beam)→전후, joint_z→상하.
  두 축 모두 프레임 안으로 들어가게 부호 정렬. sweep 4포즈 전부 프레임 내
- voron24_params.xacro: 조인트 origin 을 확정 영점으로 갱신
  (jz_z 0.2145→0.1707, jx/noz 등). contract_check PASS
- JointStateSubscriber: 링크/조인트 바인딩 리팩터 + AxisFromDrive body→b 버그픽스
- Editor 툴(콜리전 생성·측정)·실제 OBJ 에셋·RosMessages meta 추가

※ cad/working/collider(stl) 의 STL 콜리전 메시는 git-lfs 미설치로 이번 커밋 제외.
  lfs 설치 후 별도 커밋 예정.

Co-Authored-By: Claude Opus 4.8 <noreply@anthropic.com>

File: ros2_ws/src/voron24_description/urdf/voron24_params.xacro (robot description, xacro)
@@ -29,23 +29,30 @@
        ========================================================== -->
   <!-- joint_z : base_link -> z_gantry (prismatic, axis 0 0 1)
-       joint_z=0 일 때 노즐이 베드 상면에 닿는다.
-       측정: 갠트리 Y익스트루전 하면의 Z 높이 -->
+       측정: Unity Voron24Twin 씬의 확정 영점(2026-08-18) z_gantry 링크 원점 Y.
+       ※ 이 영점에서 노즐은 베드 상면보다 약 79mm 위에 있다(Z 파킹 갭).
+         계약의 "joint_z=0 → 노즐이 베드 상면에 닿는다" 를 엄격히 맞추려면
+         jz_z 를 0.079 낮춰(≈0.0917) 야 하나, 사용자가 현재 포즈를 영점으로 확정.
+         → Z 홈 캘리브레이션은 별도 결정 사항. -->
   <xacro:property name="jz_x" value="0.0"/>
   <xacro:property name="jz_y" value="0.0"/>
-  <xacro:property name="jz_z" value="0.2145"/>      <!-- (추정) -->
+  <xacro:property name="jz_z" value="0.1707"/>      <!-- CAD 씬 확정 영점 (2026-08-18) -->
   <!-- joint_y : z_gantry -> x_beam (prismatic, axis 0 1 0)
-       joint_y=0 일 때 X빔이 최전방(베드 Y=0 라인) -->
+       joint_y=0 일 때 X빔이 최전방(베드 Y=0 라인).
+       CAD 씬 확정 영점(2026-08-18)에서 계측. 기존 추정치와 거의 일치. -->
   <xacro:property name="jy_x" value="0.0"/>
-  <xacro:property name="jy_y" value="-0.125"/>      <!-- (추정) -->
-  <xacro:property name="jy_z" value="0.012"/>       <!-- (추정) -->
+  <xacro:property name="jy_y" value="-0.125"/>      <!-- CAD 씬 (2026-08-18) -->
+  <xacro:property name="jy_z" value="0.010"/>       <!-- CAD 씬 (2026-08-18) -->
   <!-- joint_x : x_beam -> toolhead (prismatic, axis 1 0 0)
-       joint_x=0 일 때 툴헤드가 최좌측(베드 X=0 라인) -->
-  <xacro:property name="jx_x" value="-0.125"/>      <!-- (추정) -->
-  <xacro:property name="jx_y" value="0.0"/>
-  <xacro:property name="jx_z" value="0.0"/>
-  <!-- nozzle : toolhead -> nozzle (fixed) — TCP -->
-  <xacro:property name="noz_x" value="0.0"/>
-  <xacro:property name="noz_y" value="0.0085"/>     <!-- (추정) -->
-  <xacro:property name="noz_z" value="-0.0520"/>    <!-- (추정) -->
+       joint_x=0 일 때 툴헤드가 최좌측(베드 X=0 라인).
+       CAD 씬 확정 영점(2026-08-18)에서 계측. jx_x 는 툴헤드가 빔을 따라
+       놓인 위치(이동축 방향), jx_y/jx_z 는 캐리지 장착 오프셋. -->
+  <xacro:property name="jx_x" value="-0.139"/>      <!-- CAD 씬 (2026-08-18) -->
+  <xacro:property name="jx_y" value="0.0565"/>     <!-- CAD 씬 (2026-08-18) -->
+  <xacro:property name="jx_z" value="0.0254"/>     <!-- CAD 씬 (2026-08-18) -->
+  <!-- nozzle : toolhead -> nozzle (fixed) — TCP
+       CAD 씬 확정 영점(2026-08-18)에서 계측한 toolhead 링크 원점 → 노즐 TCP 오프셋. -->
+  <xacro:property name="noz_x" value="0.0126"/>    <!-- CAD 씬 (2026-08-18) -->
+  <xacro:property name="noz_y" value="-0.0184"/>   <!-- CAD 씬 (2026-08-18) -->
+  <xacro:property name="noz_z" value="-0.0628"/>   <!-- CAD 씬 (2026-08-18) -->
   <!-- bed_origin : base_link -> bed_origin (fixed)
        G-code (0,0,0). 베드 상면의 좌전방 프린트 원점 코너. -->
